File: Subaru.kicad_pcb (KiCad board)
At the start: 2 copper layers, 52.7 x 43.8 mm, 30 parts, among them J1 DB15_Male, J2 SYNC_SEL, J3 USB_C_Power, J4 SYNC_OUT_SEL, J5 Mini-DIN-4-S, J7 DB15_Female_HighDensity, U1 74HC86, U2 BH7236AF, Y1 3.579545M

Commit message: feedback from the 1st lot
- modify footprint for S connector
- add a comment on noise in the circuit
Changed lines of the file:
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@@
     )
     (fp_line (start 7 -8.5) (end 7 4) (layer "F.SilkS") (width 0.15))
-    (fp_line (start -7 -8.5) (end -7 4) (layer "F.SilkS") (width 0.15))
     (fp_line (start -7 4) (end 7 4) (layer "F.SilkS") (width 0.15))
     (fp_line (start -7 -8.5) (end 7 -8.5) (layer "F.SilkS") (width 0.15))
+    (fp_line (start -7 -8.5) (end -7 4) (layer "F.SilkS") (width 0.15))
+    (fp_line (start 0 2.5) (end 0 -8.5) (layer "F.CrtYd") (width 0.15))
+    (fp_line (start 0 0) (end -6.75 0) (layer "F.CrtYd") (width 0.15))
     (fp_line (start 6.75 -3.5) (end 6.75 0.25) (layer "F.CrtYd") (width 0.15))
+    (fp_line (start -1 -3.8) (end 1 -3.8) (layer "F.CrtYd") (width 0.15))
+    (fp_line (start 3.4 -0.4) (end 3.4 2.9) (layer "F.CrtYd") (width 0.15))
+    (fp_line (start -6.75 -3.5) (end -6.75 0.25) (layer "F.CrtYd") (width 0.15))
+    (fp_line (start -5 2.5) (end 5 2.5) (layer "F.CrtYd") (width 0.15))
     (fp_line (start 0 0) (end 6.75 0) (layer "F.CrtYd") (width 0.15))
     (fp_line (start -3.4 -0.4) (end -3.4 2.9) (layer "F.CrtYd") (width 0.15))
     (fp_line (start -7 -3) (end 7 -3) (layer "F.CrtYd") (width 0.15))
-    (fp_line (start 0 2.5) (end 0 -8.5) (layer "F.CrtYd") (width 0.15))
-    (fp_line (start 0 0) (end -6.75 0) (layer "F.CrtYd") (width 0.15))
-    (fp_line (start -5 2.5) (end 5 2.5) (layer "F.CrtYd") (width 0.15))
-    (fp_line (start 3.4 -0.4) (end 3.4 2.9) (layer "F.CrtYd") (width 0.15))
-    (fp_line (start -6.75 -3.5) (end -6.75 0.25) (layer "F.CrtYd") (width 0.15))
-    (fp_line (start -1 -3.8) (end 1 -3.8) (layer "F.CrtYd") (width 0.15))
-    (pad "" thru_hole oval (at 6.75 -3) (size 1.5 4) (drill oval 0.5 3) (layers *.Cu *.Mask))
-    (pad "" thru_hole oval (at -6.75 -3) (size 1.5 4) (drill oval 0.5 3) (layers *.Cu *.Mask))
+    (pad "" thru_hole oval (at 6.75 -3) (size 1.5 4) (drill oval 0.8 3.2) (layers *.Cu *.Mask))
     (pad "" thru_hole oval (at 0 -3.8) (size 4 1.5) (drill oval 3 0.5) (layers *.Cu *.Mask))
-    (pad "1" thru_hole oval (at -3.4 0) (size 1.4 1.4) (drill oval 0.4 1) (layers *.Cu *.Mask)
+    (pad "" thru_hole oval (at -6.75 -3) (size 1.5 4) (drill oval 0.8 3.2) (layers *.Cu *.Mask))
+    (pad "1" thru_hole oval (at -3.4 0) (size 1.4 1.4) (drill oval 0.8 1) (layers *.Cu *.Mask)
       (net 8 "GND") (pintype "passive"))
-    (pad "2" thru_hole oval (at 3.4 0) (size 1.4 1.4) (drill oval 0.4 1) (layers *.Cu *.Mask)
+    (pad "2" thru_hole oval (at 3.4 0) (size 1.4 1.4) (drill oval 0.8 1) (layers *.Cu *.Mask)
       (net 8 "GND") (pintype "passive"))
-    (pad "3" thru_hole oval (at -3.4 2.4) (size 1.4 1.4) (drill oval 0.4 1) (layers *.Cu *.Mask)
+    (pad "3" thru_hole oval (at -3.4 2.4) (size 1.4 1.4) (drill oval 0.8 1) (layers *.Cu *.Mask)
       (net 32 "/S_Y") (pintype "passive"))
-    (pad "4" thru_hole oval (at 3.4 2.5) (size 1.4 1.4) (drill oval 0.4 1) (layers *.Cu *.Mask)
+    (pad "4" thru_hole oval (at 3.4 2.5) (size 1.4 1.4) (drill oval 0.8 1) (layers *.Cu *.Mask)
       (net 33 "/S_C") (pintype "passive"))
   )
